File: ESC carrier board test 1.kicad_pcb (KiCad board)
At the start: 2 copper layers, 100 x 97.5 mm, 8 parts, among them J1 Conn_01x04_Pin, J3 Conn_01x04_Pin, J4 Conn_01x04_Pin, U1 ESC, U2 ESC, U3 ESC

Commit message: Add files via upload
Parts:
- moved J3 3.31 mm to (165.9, 106.0)
- moved U3 1.59 mm to (132.2, 123.6)
- moved J4 0.57 mm to (165.8, 117.6)
- moved U2 0.41 mm to (112.2, 123.6)
Connections:
- J1 pad 1: /sGP37 -> /sGP10
- J1 pad 2: /sGP38 -> /sGP10
- U2 pad S: /sGP38 -> /sGP10
- U3 pad S: /sGP37 -> /sGP8
- U7 pad 16: /sGP37 -> unconnected-(U7-GP37-Pad16)
- U7 pad 17: /sGP38 -> unconnected-(U7-GP38-Pad17)
- U7 pad 19: /signalGP39 -> unconnected-(U7-GP39-Pad19)
- U7 pad 2: unconnected-(U7-GP12-Pad2) -> Net-(J3-Pin_4)
- U7 pad 24: Net-(J4-Pin_2) -> unconnected-(U7-GP1-Pad24)
- U7 pad 25: Net-(J4-Pin_3) -> Net-(J4-Pin_2)
- U7 pad 26: Net-(J4-Pin_4) -> Net-(J4-Pin_3)
- U7 pad 28: Net-(J3-Pin_1) -> unconnected-(U7-GND-Pad28)
- U7 pad 29: Net-(J3-Pin_2) -> Net-(J4-Pin_4)
- U7 pad 31: Net-(J3-Pin_3) -> unconnected-(U7-GP7-Pad31)
- U7 pad 32: Net-(J3-Pin_4) -> /sGP8
- U7 pad 35: unconnected-(U7-GP10-Pad35) -> /sGP10
- U7 pad 5: unconnected-(U7-GP14-Pad5) -> Net-(J3-Pin_3)
- U7 pad 7: unconnected-(U7-GP16-Pad7) -> Net-(J3-Pin_2)
- U7 pad 8: unconnected-(U7-GND-Pad8) -> Net-(J3-Pin_1)
Other:
- outline, holes or cut-outs redrawn
