File: ESC carrier board test 1.kicad_sch (KiCad schematic)
At the start: 11 parts, among them J1 Conn_01x04_Pin, J3 Conn_01x04_Pin, J4 Conn_01x04_Pin, U1 ESC, U2 ESC, U3 ESC

Commit message: Add files via upload
Connections:
- net signalGP39: no longer U7.19 (GP39)
- net at J4.2 (Pin_2): now also U7.25 (GP2); no longer U7.24 (GP1)
- net at J4.3 (Pin_3): now also U7.26 (GP4); no longer U7.25 (GP2)
- net at J4.4 (Pin_4): now also U7.29 (GP6); no longer U7.26 (GP4)
- net at J3.1 (Pin_1): now also U7.8 (GND); no longer U7.28 (GND)
- net at J3.2 (Pin_2): now also U7.7 (GP16); no longer U7.29 (GP6)
- net at J3.3 (Pin_3): now also U7.5 (GP14); no longer U7.31 (GP7)
- net at J3.4 (Pin_4): now also U7.2 (GP12); no longer U7.32 (GP8)
- net sGP10: now reaches U7.35 (GP10)
- net sGP10: now also J1.1 (Pin_1), J1.2 (Pin_2), U2.S
- removed net sGP37: J1.1 (Pin_1), U3.S, U7.16 (GP37)
- removed net sGP38: J1.2 (Pin_2), U2.S, U7.17 (GP38)
- new net sGP8: U3.S, U7.32 (GP8)
Other:
- moved on the sheet: U7
Changed lines of the file:
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@@
 (kicad_sch (version 20230121) (generator eeschema)
   (paper "A4")
-  (wire (pts (xy 222.25 142.24) (xy 232.41 142.24))
-    (stroke (width 0) (type default))
-  )
-  (wire (pts (xy 260.35 119.38) (xy 260.35 116.84))
+  (wire (pts (xy 264.16 134.62) (xy 264.16 132.08))
+    (stroke (width 0) (type default))
+  )
+  (wire (pts (xy 231.14 114.3) (xy 231.14 106.68))
     (stroke (width 0) (type default))
   )
@@
     (stroke (width 0) (type default))
   )
-  (wire (pts (xy 255.27 127) (xy 264.16 127))
+  (wire (pts (xy 237.49 111.76) (xy 233.68 111.76))
     (stroke (width 0) (type default))
   )
@@
     (stroke (width 0) (type default))
   )
-  (wire (pts (xy 264.16 119.38) (xy 260.35 119.38))
-    (stroke (width 0) (type default))
-  )
   (wire (pts (xy 138.43 72.39) (xy 138.43 88.9))
     (stroke (width 0) (type default))
   )
-  (wire (pts (xy 257.81 121.92) (xy 264.16 121.92))
-    (stroke (width 0) (type default))
-  )
-  (wire (pts (xy 269.24 132.08) (xy 255.27 132.08))
+  (wire (pts (xy 269.24 137.16) (xy 261.62 137.16))
     (stroke (width 0) (type default))
   )
@@
     (stroke (width 0) (type default))
   )
-  (wire (pts (xy 255.27 119.38) (xy 257.81 119.38))
-    (stroke (width 0) (type default))
-  )
   (wire (pts (xy 170.18 88.9) (xy 170.18 72.39))
     (stroke (width 0) (type default))
   )
-  (wire (pts (xy 269.24 139.7) (xy 255.27 139.7))
-    (stroke (width 0) (type default))
-  )
-  (wire (pts (xy 269.24 134.62) (xy 255.27 134.62))
+  (wire (pts (xy 269.24 139.7) (xy 260.35 139.7))
+    (stroke (width 0) (type default))
+  )
+  (wire (pts (xy 266.7 124.46) (xy 266.7 132.08))
     (stroke (width 0) (type default))
   )
@@
     (stroke (width 0) (type default))
   )
-  (wire (pts (xy 257.81 119.38) (xy 257.81 121.92))
+  (wire (pts (xy 236.22 106.68) (xy 236.22 101.6))
+    (stroke (width 0) (type default))
+  )
+  (wire (pts (xy 261.62 134.62) (xy 260.35 134.62))
     (stroke (width 0) (type default))
   )
@@
     (stroke (width 0) (type default))
   )
+  (wire (pts (xy 269.24 132.08) (xy 266.7 132.08))
+    (stroke (width 0) (type default))
+  )
   (wire (pts (xy 162.56 88.9) (xy 165.1 88.9))
     (stroke (width 0) (type default))
@@
     (stroke (width 0) (type default))
   )
+  (wire (pts (xy 269.24 134.62) (xy 264.16 134.62))
+    (stroke (width 0) (type default))
+  )
   (wire (pts (xy 120.65 127) (xy 120.65 130.81))
     (stroke (width 0) (type default))
   )
-  (wire (pts (xy 223.52 127) (xy 232.41 127))
+  (wire (pts (xy 223.52 127) (xy 237.49 127))
+    (stroke (width 0) (type default))
+  )
+  (wire (pts (xy 237.49 139.7) (xy 232.41 139.7))
+    (stroke (width 0) (type default))
+  )
+  (wire (pts (xy 264.16 132.08) (xy 260.35 132.08))
+    (stroke (width 0) (type default))
+  )
+  (wire (pts (xy 237.49 114.3) (xy 231.14 114.3))
     (stroke (width 0) (type default))
   )
@@
     (stroke (width 0) (type default))
   )
-  (wire (pts (xy 255.27 124.46) (xy 264.16 124.46))
+  (wire (pts (xy 261.62 137.16) (xy 261.62 134.62))
+    (stroke (width 0) (type default))
+  )
+  (wire (pts (xy 236.22 101.6) (xy 231.14 101.6))
     (stroke (width 0) (type default))
   )
@@
     (stroke (width 0) (type default))
   )
-  (wire (pts (xy 269.24 137.16) (xy 255.27 137.16))
+  (wire (pts (xy 233.68 111.76) (xy 233.68 104.14))
+    (stroke (width 0) (type default))
+  )
+  (wire (pts (xy 237.49 106.68) (xy 236.22 106.68))
+    (stroke (width 0) (type default))
+  )
+  (wire (pts (xy 233.68 104.14) (xy 231.14 104.14))
+    (stroke (width 0) (type default))
+  )
+  (wire (pts (xy 266.7 124.46) (xy 260.35 124.46))
+    (stroke (width 0) (type default))
+  )
+  (wire (pts (xy 231.14 99.06) (xy 237.49 99.06))
     (stroke (width 0) (type default))
   )
@@
     (stroke (width 0) (type default))
   )
-  (wire (pts (xy 255.27 116.84) (xy 260.35 116.84))
+  (wire (pts (xy 260.35 99.06) (xy 255.27 99.06))
     (stroke (width 0) (type default))
   )
@@
     (effects (font (size 1.27 1.27)) (justify left bottom))
   )
-  (label "sGP37" (at 243.84 151.13 0) (fields_autoplaced)
+  (label "sGP10" (at 243.84 151.13 0) (fields_autoplaced)
     (effects (font (size 1.27 1.27)) (justify left bottom))
   )
@@
     (effects (font (size 1.27 1.27)) (justify left bottom))
   )
-  (label "sGP38" (at 232.41 137.16 0) (fields_autoplaced)
-    (effects (font (size 1.27 1.27)) (justify left bottom))
-  )
-  (label "sGP38" (at 165.1 127 0) (fields_autoplaced)
+  (label "sGP10" (at 260.35 109.22 0) (fields_autoplaced)
+    (effects (font (size 1.27 1.27)) (justify left bottom))
+  )
+  (label "sGP10" (at 165.1 127 0) (fields_autoplaced)
     (effects (font (size 1.27 1.27)) (justify left bottom))
   )
@@
     (effects (font (size 1.27 1.27)) (justify left bottom))
   )
-  (label "sGP37" (at 232.41 134.62 0) (fields_autoplaced)
-    (effects (font (size 1.27 1.27)) (justify left bottom))
-  )
-  (label "signalGP39" (at 222.25 142.24 0) (fields_autoplaced)
+  (label "sGP8" (at 260.35 116.84 0) (fields_autoplaced)
+    (effects (font (size 1.27 1.27)) (justify left bottom))
+  )
+  (label "signalGP39" (at 271.78 101.6 0) (fields_autoplaced)
     (effects (font (size 1.27 1.27)) (justify left bottom))
   )
@@
     (effects (font (size 1.27 1.27)) (justify left bottom))
   )
-  (label "sGP38" (at 243.84 153.67 0) (fields_autoplaced)
+  (label "sGP10" (at 243.84 153.67 0) (fields_autoplaced)
     (effects (font (size 1.27 1.27)) (justify left bottom))
   )
@@
     (effects (font (size 1.27 1.27)) (justify left bottom))
   )
-  (label "sGP37" (at 203.2 127 0) (fields_autoplaced)
+  (label "sGP8" (at 203.2 127 0) (fields_autoplaced)
     (effects (font (size 1.27 1.27)) (justify left bottom))
   )
@@
     )
   )
-  (symbol (lib_id "Connector:Conn_01x04_Pin") (at 269.24 124.46 180) (unit 1)
-    (in_bom yes) (on_board yes) (dnp no) (fields_autoplaced)
-    (property "Reference" "J3" (at 270.51 121.92 0)
-      (effects (font (size 1.27 1.27)) (justify right))
-    )
-    (property "Value" "Conn_01x04_Pin" (at 270.51 124.46 0)
-      (effects (font (size 1.27 1.27)) (justify right))
-    )
-    (property "Footprint" "Connector_PinHeader_2.54mm:PinHeader_1x04_P2.54mm_Horizontal" (at 269.24 124.46 0)
-      (effects (font (size 1.27 1.27)) hide)
-    )
-    (property "Datasheet" "~" (at 269.24 124.46 0)
+  (symbol (lib_id "Connector:Conn_01x04_Pin") (at 226.06 104.14 0) (mirror x) (unit 1)
+    (in_bom yes) (on_board yes) (dnp no)
+    (property "Reference" "J3" (at 226.695 111.76 0)
+      (effects (font (size 1.27 1.27)) hide)
+    )
+    (property "Value" "Conn_01x04_Pin" (at 226.06 109.22 0)
+      (effects (font (size 1.27 1.27)) hide)
+    )
+    (property "Footprint" "Connector_PinHeader_2.54mm:PinHeader_1x04_P2.54mm_Horizontal" (at 226.06 104.14 0)
+      (effects (font (size 1.27 1.27)) hide)
+    )
+    (property "Datasheet" "~" (at 226.06 104.14 0)
       (effects (font (size 1.27 1.27)) hide)
     )
@@
     )
   )
-  (symbol (lib_id "Kelpie_Library:ESP32-S3-Pico") (at 243.84 113.03 0) (unit 1)
-    (in_bom yes) (on_board yes) (dnp no) (fields_autoplaced)
-    (property "Reference" "U7" (at 243.84 92.71 0)
-      (effects (font (size 1.27 1.27)))
-    )
-    (property "Value" "~" (at 243.84 113.03 0)
-      (effects (font (size 1.27 1.27)))
-    )
-    (property "Footprint" "Kelpie_Default:ESP32-S3-Pico" (at 243.84 113.03 0)
-      (effects (font (size 1.27 1.27)) hide)
-    )
-    (property "Datasheet" "" (at 243.84 113.03 0)
-      (effects (font (size 1.27 1.27)) hide)
-    )
+  (symbol (lib_id "Kelpie_Library:ESP32-S3-Pico") (at 248.92 113.03 0) (unit 1)
+    (in_bom yes) (on_board yes) (dnp no) (fields_autoplaced)
+    (property "Reference" "U7" (at 248.92 92.71 0)
+      (effects (font (size 1.27 1.27)))
+    )
+    (property "Value" "~" (at 248.92 113.03 0)
+      (effects (font (size 1.27 1.27)))
+    )
+    (property "Footprint" "Kelpie_Default:ESP32-S3-Pico" (at 248.92 113.03 0)
+      (effects (font (size 1.27 1.27)) hide)
+    )
+    (property "Datasheet" "" (at 248.92 113.03 0)
+      (effects (font (size 1.27 1.27)) hide)
+    )
