File: ESC carrier board/ESC carrier board.kicad_pcb (KiCad board)
At the start: 2 copper layers, 100 x 97.5 mm, 8 parts, among them J1 Conn_01x04_Pin, J3 Conn_01x04_Pin, J4 Conn_01x04_Pin, U1 ESC, U2 ESC, U3 ESC

Commit message: Modified board
Parts:
- removed U1, U3: ESC, ESC carrier board test 1:ESC
- added J5: Conn_01x04_Pin, Connector_PinHeader_2.54mm:PinHeader_1x04_P2.54mm_Horizontal, B.Cu at (166.4, 118.1)
- added JP1: Jumper_3_Open, Jumper:SolderJumper-3_P1.3mm_Open_RoundedPad1.0x1.5mm, F.Cu at (153.7, 144.8)
- added JP2: Jumper_3_Open, Jumper:SolderJumper-3_P1.3mm_Open_RoundedPad1.0x1.5mm, F.Cu at (161.3, 144.8)
- added JP3: Jumper_2_Bridged, Jumper:SolderJumper-2_P1.3mm_Open_RoundedPad1.0x1.5mm, F.Cu at (167.6, 145.4)
- added JP4: Jumper_2_Bridged, Jumper:SolderJumper-2_P1.3mm_Open_RoundedPad1.0x1.5mm, F.Cu at (170.2, 145.4)
- added SW1: SW_DPDT_x2, Kelpie_Default:CUI-Switch-SMD, F.Cu at (152.4, 133.3)
- added U4: ESC, ESC-carrier:ESC, F.Cu at (113.7, 120.0)
- added U6: ESC, ESC-carrier:ESC, F.Cu at (134.0, 120.0)
- J1: value Conn_01x04_Pin -> ~; footprint Connector_PinHeader_2.54mm:PinHeader_1x04_P2.54mm_Horizontal -> 2024-backplane:MR60PW-M_X3
- J2: footprint ESC carrier board test 1:MR60PW-M_X3 -> 2024-backplane:CardEdge_2x10
- U2: footprint ESC carrier board test 1:ESC -> ESC-carrier:ESC
- moved J1 56.8 mm to (109.9, 147.4)
- moved J2 38.9 mm to (149.6, 158.2)
- moved U2 19.1 mm to (93.4, 120.0)
- moved J4 17.0 mm to (166.4, 134.6)
- moved U7 4.22 mm to (151.1, 87.6)
- moved J3 0.88 mm to (166.4, 106.7)
Connections:
- J1 pad 1: /sGP10 -> unconnected-(J1A-48V-Pad1)
- J1 pad 2: /sGP10 -> GND
- J1 pad 3: /signalGP39 -> GND
- J1 pad 4: /sg -> /PESC1
- J2 pad 1: unconnected-(J2A-A-Pad1) -> sGND
- J2 pad 2: /GND -> Net-(J2-TX0/SDA0)
- J2 pad 3: /GND -> Net-(J2-RX0/SCL0)
- J2 pad 4: /PESC1 -> sGND
- J2 pad 5: /PESC2 -> Net-(J2-TX1/SDA1)
- J2 pad 6: /PESC3 -> Net-(J2-RX1/SCL1)
- J2 pad 7: unconnected-(J2C-A-Pad7) -> sGND
- J2 pad 8: /GND -> Net-(J2-TX2/SDA2)
- J2 pad 9: /5v -> Net-(J2-RX2/SCL2)
- J4 pad 1: Net-(J4-Pin_1) -> /sg
- J4 pad 2: Net-(J4-Pin_2) -> /sGP6
- J4 pad 3: Net-(J4-Pin_3) -> /sGP7
- J4 pad 4: Net-(J4-Pin_4) -> /sGP8
- U2 pad +: /PESC2 -> /PESC1
- U2 pad -: /GND -> GND
- U2 pad S: /sGP10 -> /sGP8
- U7 pad 1: unconnected-(U7-GP11-Pad1) -> TX0
- U7 pad 10: unconnected-(U7-GP18-Pad10) -> /sGP7
- U7 pad 11: unconnected-(U7-GP33-Pad11) -> /sGP8
- U7 pad 18: /GND -> GND
- U7 pad 2: Net-(J3-Pin_4) -> RX0
- U7 pad 21: unconnected-(U7-GP42-Pad21) -> Net-(J5-Pin_2)
- U7 pad 22: unconnected-(U7-GP41-Pad22) -> Net-(J5-Pin_3)
- U7 pad 23: Net-(J4-Pin_1) -> Net-(J5-Pin_1)
- U7 pad 24: unconnected-(U7-GP1-Pad24) -> Net-(J5-Pin_4)
- U7 pad 25: Net-(J4-Pin_2) -> unconnected-(U7-GP19-Pad25)
- U7 pad 26: Net-(J4-Pin_3) -> SDA0
- U7 pad 27: unconnected-(U7-GP5-Pad27) -> SCL0
- U7 pad 29: Net-(J4-Pin_4) -> unconnected-(U7-GP22-Pad29)
- U7 pad 31: unconnected-(U7-GP7-Pad31) -> SDA1
- U7 pad 32: /sGP8 -> SCL1
- U7 pad 35: /sGP10 -> unconnected-(U7-ADC_VREF-Pad35)
- U7 pad 5: Net-(J3-Pin_3) -> Net-(J3-Pin_4)
- U7 pad 6: unconnected-(U7-GP15-Pad6) -> Net-(J3-Pin_3)
- U7 pad 9: unconnected-(U7-GP17-Pad9) -> /sGP6
Routing:
- net SCL1: track 0.00 -> 58.5 mm, vias 0 -> 1
- net SDA1: track 0.00 -> 53.2 mm, vias 0 -> 1
- net Net-(J3-Pin_1): track 0.00 -> 2.68 mm
- net Net-(J3-Pin_2): track 0.00 -> 2.09 mm
- net Net-(J5-Pin_3): track 0.00 -> 1.27 mm
- net Net-(J5-Pin_2): track 0.00 -> 0.64 mm
Other:
- outline, holes or cut-outs redrawn
