File: template-card/template-card.kicad_pcb (KiCad board)
At the start: 2 copper layers, 2 parts, among them J1 Conn_01x10_Pin

Commit message: blergh
Parts:
- added SW1: SW_DPDT_x2, 2024-backplane:SW_CUI_DPDT, F.Cu at (180.4, 102.1)
- moved J2 17.5 mm to (125.1, 130.8)
- moved J1 17.1 mm to (170.6, 140.0)
Connections:
- J1 pad 1: unconnected-(J1-Pin_1-Pad1) -> GND1
- J1 pad 10: unconnected-(J1-Pin_10-Pad10) -> GND1
- J1 pad 2: unconnected-(J1-Pin_2-Pad2) -> /tx0/sda0
- J1 pad 3: unconnected-(J1-Pin_3-Pad3) -> /rx0/scl0
- J1 pad 4: unconnected-(J1-Pin_4-Pad4) -> GND1
- J1 pad 5: unconnected-(J1-Pin_5-Pad5) -> /tx1/sda1
- J1 pad 6: unconnected-(J1-Pin_6-Pad6) -> /rx1/scl1
- J1 pad 7: unconnected-(J1-Pin_7-Pad7) -> GND1
- J1 pad 8: unconnected-(J1-Pin_8-Pad8) -> /tx2/sda2
- J1 pad 9: unconnected-(J1-Pin_9-Pad9) -> /rx2/scl2
- J2 pad 1: unconnected-(J2A-A-Pad1) -> /48v
- J2 pad 2: unconnected-(J2A-B-Pad2) -> /24v
- J2 pad 3: unconnected-(J2A-C-Pad3) -> GND2
- J2 pad 4: unconnected-(J2B-A-Pad4) -> /12v
- J2 pad 5: unconnected-(J2B-B-Pad5) -> /12v
- J2 pad 6: unconnected-(J2B-C-Pad6) -> /12v
- J2 pad 7: unconnected-(J2C-A-Pad7) -> GND2
- J2 pad 8: unconnected-(J2C-B-Pad8) -> /5v
- J2 pad 9: unconnected-(J2C-C-Pad9) -> GND2
Other:
- board outline added: 27.6 x 8 mm

Commit message: template finished
Parts:
- moved J2 39.2 mm to (122.1, 91.8)
- moved J1 36.0 mm to (172.2, 104.0)
- moved SW1 25.9 mm to (177.9, 76.3)
Other:
- board size 27.6 x 8 mm -> 111.8 x 83 mm
Changed lines of the file:
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@@
   (net 16 "/scl")
   (footprint "2024-backplane:MR60PW-M_X3" (layer "F.Cu")
-    (at 125.1 130.85)
+    (at 122.13 91.76)
     (property "Sheetfile" "template-card.kicad_sch")
     (property "Sheetname" "")
@@
   )
   (footprint "2024-backplane:SW_CUI_DPDT" (layer "F.Cu")
-    (at 180.38 102.06)
+    (at 177.925 76.3)
     (property "Sheetfile" "template-card.kicad_sch")
     (property "Sheetname" "")
@@
   )
   (footprint "2024-backplane:CardEdge_2x10" (layer "F.Cu")
-    (at 170.62 140)
+    (at 172.22 104)
     (property "Sheetfile" "template-card.kicad_sch")
     (property "Sheetname" "")
@@
       (net 1 "GND1") (pinfunction "Pin_10") (pintype "passive") (thermal_bridge_angle 45))
   )
-  (gr_line (start 195.9 144.042) (end 168.26 144.042)
+  (gr_line (start 197.5 108.042) (end 169.86 108.042)
     (stroke (width 0.1) (type default)) (layer "Edge.Cuts"))
-  (gr_line (start 195.9 144.042) (end 195.9 136)
+  (gr_line (start 197.5 108.042) (end 197.5 100)
     (stroke (width 0.1) (type default)) (layer "Edge.Cuts"))
-  (gr_line (start 168.26 144.042) (end 168.26 136)
+  (gr_line (start 85.68 100) (end 85.68 25)
+    (stroke (width 0.1) (type default)) (layer "Edge.Cuts"))
+  (gr_line (start 85.68 25) (end 197.5 25)
+    (stroke (width 0.1) (type default)) (layer "Edge.Cuts"))
+  (gr_line (start 169.86 100) (end 85.68 100)
+    (stroke (width 0.1) (type default)) (layer "Edge.Cuts"))
+  (gr_line (start 197.5 100) (end 197.5 25)
+    (stroke (width 0.1) (type default)) (layer "Edge.Cuts"))
+  (gr_line (start 169.86 108.042) (end 169.86 100)
     (stroke (width 0.1) (type default)) (layer "Edge.Cuts"))
 )
