File: 12V/Bus 1/bus1.kicad_sch (KiCad schematic)
At the start: 4 parts, among them J1 Conn_01x10_Pin, SW1 SW_DPDT_x2

Commit message: Completed Prelim Board Layout
Parts:
- removed SW1: SW_DPDT_x2, 2024-backplane:SW_CUI_DPDT, symbol Switch:SW_DPDT_x2
Connections:
- net GND1: no longer PS1.2 (On/Off)
- net GND2: now also PS1.2 (On/Off)
- net 12v renamed 12v_1
- net 12v_1: no longer J2.5 (12V), J2.6 (12V)
- net 24v: no longer names the net of J2.7 (24V)
- net 5v: no longer names the net of J2.9 (5V)
- net rx0/scl0: no longer names the net of J1.3 (RX0/SCL0)
- net rx1/scl1: no longer names the net of J1.6 (RX1/SCL1)
- net rx2/scl2: no longer names the net of J1.9 (RX2/SCL2)
- net tx0/sda0: no longer names the net of J1.2 (TX0/SDA0)
- net tx1/sda1: no longer names the net of J1.5 (TX1/SDA1)
- net tx2/sda2: no longer names the net of J1.8 (TX2/SDA2)
- no-connect marks 6 -> 10
Other:
- moved on the sheet: PS1
