File: 12V/Bus 1/bus1.kicad_pcb (KiCad board)
At the start: 2 copper layers, 111.8 x 83 mm, 3 parts, among them J1 Conn_01x10_Pin, SW1 SW_DPDT_x2

Commit message: Completed Prelim Board Layout
Parts:
- removed SW1: SW_DPDT_x2, 2024-backplane:SW_CUI_DPDT
- added PS1: DCE0133V2NBC, 2024-power:Murata DCE0133V2NBC, F.Cu at (92.1, 62.8)
Connections:
- J1 pad 2: /tx0/sda0 -> unconnected-(J1-TX0/SDA0-Pad2)
- J1 pad 3: /rx0/scl0 -> unconnected-(J1-RX0/SCL0-Pad3)
- J1 pad 5: /tx1/sda1 -> unconnected-(J1-TX1/SDA1-Pad5)
- J1 pad 6: /rx1/scl1 -> unconnected-(J1-RX1/SCL1-Pad6)
- J1 pad 8: /tx2/sda2 -> unconnected-(J1-TX2/SDA2-Pad8)
- J1 pad 9: /rx2/scl2 -> unconnected-(J1-RX2/SCL2-Pad9)
- J2 pad 2: /24v -> GND2
- J2 pad 4: /12v -> /12v_1
- J2 pad 5: /12v -> unconnected-(J2B-12V-Pad5)
- J2 pad 6: /12v -> unconnected-(J2B-12V-Pad6)
- J2 pad 7: GND2 -> unconnected-(J2C-24V-Pad7)
- J2 pad 8: /5v -> GND2
- J2 pad 9: GND2 -> unconnected-(J2C-5V-Pad9)
Routing:
- net GND1: track 0.00 -> 26.6 mm
- net GND2: vias 0 -> 188
- net /48v: vias 0 -> 43
- net /12v_1: vias 0 -> 137
- added copper zone on B.Cu, net /12v_1
- added copper zone on F.Cu, net /12v_1
- added copper zone on B.Cu, net /48v
- added copper zone on F.Cu, net /48v
- added copper zone on B.Cu, net GND2
- added copper zone on F.Cu, net GND2
Other:
- board size 111.8 x 83 mm -> 111.8 x 53 mm

Commit message: JLC Design Constraints
Routing:
- net GND2: vias 188 -> 191
- net /12v_1: vias 137 -> 134
