File: 12V/Bus3/bus3.kicad_pcb (KiCad board)
At the start: 2 copper layers, 111.8 x 53 mm, 3 parts, among them J1 Conn_01x10_Pin

Commit message: JLC Design Constraints
Routing:
- net GND2: vias 188 -> 189
- net /12v_3: vias 149 -> 147
